Commit message: make odom work w articubot

File: alffybot/install/alffy_description/share/alffy_description/urdf/alffy_gazebo.xacro (robot description, xacro)
@@ -37,9 +37,11 @@
     <maxVel>1.0</maxVel>
   </gazebo>
-  <!-- ROS 2 Control -->
+<!--
+ ROS 2 Control  -->
   <gazebo>
     <xacro>
-      <plugin filename="libgz_ros2_control-system.so" name="gz_ros2_control::GazeboSimROS2ControlPlugin">
+      <plugin filename="libgz_ros2_control-system" name="gz_ros2_control::GazeboSimROS2ControlPlugin">
         <parameters>$(find alffy_controller)/config/alffy_controllers.yaml</parameters>
+        <controller_manager_prefix_node_name>controller_manager</controller_manager_prefix_node_name>
       </plugin>
     </xacro>

File: alffybot/install/alffy_description/share/alffy_description/urdf/alffy_ros2_control.xacro (robot description, xacro)
@@ -16,5 +16,5 @@
             <state_interface name="velocity" />
         </joint>
-        <joint name="wheel_left_joint">
+        <joint name="wheel_left_jointto become available...">
             <command_interface name="velocity">
               <param name="min">-1</param>
@@ -25,3 +25,11 @@
         </joint>
     </ros2_control>
+    <!-- ROS 2 Control -->
+        <gazebo>
+            <!-- <plugin filename="libgz_ros2_control-system.so" name="gz_ros2_control::GazeboSimROS2ControlPlugin"> -->
+            <plugin name="gz_ros2_control::GazeboSimROS2ControlPlugin" filename="libgz_ros2_control-system">
+                <parameters>$(find alffy_controller)/config/alffy_controllers.yaml</parameters>
+                <controller_manager_prefix_node_name>controller_manager</controller_manager_prefix_node_name>
+            </plugin>
+        </gazebo>
 </robot>

File: alffybot/src/alffy_description/urdf/alffy_ros2_control.xacro (robot description, xacro)
@@ -16,5 +16,5 @@
             <state_interface name="velocity" />
         </joint>
-        <joint name="wheel_left_joint">
+        <joint name="wheel_left_jointto become available...">
             <command_interface name="velocity">
               <param name="min">-1</param>
@@ -25,3 +25,13 @@
         </joint>
     </ros2_control>
+    <!-- ROS 2 Control -->
+        <gazebo>
+            <xacro>
+            <!-- <plugin filename="libgz_ros2_control-system.so" name="gz_ros2_control::GazeboSimROS2ControlPlugin"> -->
+                <plugin name="gz_ros2_control::GazeboSimROS2ControlPlugin" filename="libgz_ros2_control-system">
+                    <parameters>$(find alffy_controller)/config/alffy_controllers.yaml</parameters>
+                    <controller_manager_prefix_node_name>controller_manager</controller_manager_prefix_node_name>
+                </plugin>
+            </xacro>
+        </gazebo>
 </robot>
