Commit message: urdf with straight plate and castor wheel on point

File: alfred_ws/src/alfred_body/description/robot_core.xacro (robot description, xacro)
@@ -208,3 +208,30 @@
         <mu2 value="0.000000000000000001"/>
     </gazebo>
+    <!-- Top Plate -->
+    <joint name="top_plate_joint" type="fixed">
+        <parent link="chassis"/>
+        <child link="top_plate"/>
+        <origin xyz="0 0 ${-wheel_offset_z+chassis_height}"/>
+    </joint>
+    <link name="top_plate">
+        <visual>
+            <origin xyz="0 0 0.480"/>
+            <geometry>
+                <box size="0.002 ${chassis_width} 0.960"/>
+            </geometry>
+            <material name="orange"/>
+        </visual>
+        <collision>
+            <origin xyz="0 0 0.480"/>
+            <geometry>
+                <box size="0.002 ${chassis_width} 0.960"/>
+            </geometry>
+        </collision>
+        <xacro:inertial_box mass="0.005" x="0.002" y="${chassis_width}" z="0.960">
+            <origin xyz="0 0 0.480" rpy="0 0 0"/>
+        </xacro:inertial_box>
+    </link>
+    <gazebo reference="chassis">
+        <material>Gazebo/White</material>
+    </gazebo>
 </robot>

File: alfred_ws/src/alfred_body/description/robot_measurements.xacro (robot description, xacro)
@@ -12,9 +12,9 @@
     <xacro:property name="wheel_offset_y" value="0.280"/>
     <xacro:property name="wheel_offset_z" value="0.01"/> <!-- To be changed-->
-    <xacro:property name="caster_wheel_radius" value="0.01"/>
+    <xacro:property name="caster_wheel_radius" value="0.03"/>
     <xacro:property name="caster_wheel_mass" value="0.01"/>
     <xacro:property name="caster_wheel_offset_x" value="0.185"/>
     <xacro:property name="caster_wheel_offset_y" value="0.235"/>
-    <xacro:property name="caster_wheel_offset_z" value="${wheel_offset_z - wheel_radius + caster_wheel_radius}"/>
+    <xacro:property name="caster_wheel_offset_z" value="${-wheel_offset_z + wheel_radius - caster_wheel_radius}"/>
     <!-- Some additional properties -->
     <material name="white">

Commit message: not sure what is changed, commiting to start a new session

File: alfred_ws/src/alfred_body/description/robot_core.xacro (robot description, xacro)
@@ -235,3 +235,30 @@
         <material>Gazebo/White</material>
     </gazebo>
+    <!-- Tray one -->
+    <!-- <joint name="tray_one_joint" type="fixed">
+        <parent link="top_plate"/>
+        <child link="top_plate"/>
+        <origin xyz="0 0 0"/>
+    </joint>
+    <link name="top_plate">
+        <visual>
+            <origin xyz="0 0 0"/>
+            <geometry>
+                <box size="0.002 ${chassis_width} 0.960"/>
+            </geometry>
+            <material name="orange"/>
+        </visual>
+        <collision>
+            <origin xyz="0 0 0"/>
+            <geometry>
+                <box size="0.002 ${chassis_width} 0.960"/>
+            </geometry>
+        </collision>
+        <xacro:inertial_box mass="0.005" x="0.002" y="${chassis_width}" z="0.960">
+            <origin xyz="0 0 0" rpy="0 0 0"/>
+        </xacro:inertial_box>
+    </link>
+    <gazebo reference="chassis">
+        <material>Gazebo/Orange</material>
+    </gazebo>  -->
 </robot>
